File: SMT-Stencil-Grid.kicad_pcb (KiCad board)
At the start: 2 copper layers, 0 parts

Commit message: Updated: 2019-02-25 10:20:51
Parts:
- added REF**: OSHW-Logo2_14.6x12mm_Copper, Symbol:OSHW-Logo2_14.6x12mm_Copper, F.Cu at (128.6, 110.7)
Other:
- board text added: "https://www.hakr.xyz"
- board text added: "https://www.iternull.com"
